File: tests/summe.kicad_sch (KiCad schematic)
At the start: 78 parts, among them J1 IDC Header, J10 OUT, J2 IN, J3 IN, J4 IN, J5 IN, J6 OUT, J7 OUT, J8 OUT, J9 OUT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

Commit message: work on reader and writer
Parts:
- C1, C2: value 22u -> 10u; footprint (none) -> Capacitor_THT:CP_Radial_D5.0mm_P2.50mm
- R28, R29, R30, R32, R34: value 500 -> 510
- RV1, RV2, RV3, RV4: footprint (none) -> elektrophon:Potentiometer_Alpha_RD901F-40-00D_Single_Vertical
